File: TallyController/EAGLE/Output Power Distro.brd (EAGLE design)
At the start: 28.9 x 29.2 mm, 6 parts

Commit message: Slim down some spacings to possibly use some 8 pin headers instead of 4x 2pin.  Fix hole drill sizes.
Parts:
- moved OUT3 3.81 mm to (14.0, 5.08)
- moved OUT4 3.81 mm to (14.0, 14.0)
- moved OUT5 3.81 mm to (14.0, 22.9)
- moved IN 3.81 mm to (7.62, 5.08)
- moved OUT1 3.81 mm to (7.62, 14.0)
- moved OUT2 3.81 mm to (7.62, 22.9)
Other:
- board size 28.9 x 29.2 mm -> 21.9 x 29.2 mm
