File: TallyController/EAGLE/tally-controller-shield-smd.brd (EAGLE design)
At the start: 101.6 x 53.3 mm, 28 parts, among them J2 Mega R3, U1 SN75174N, U2 SN75174N, U3 SN75174N

Commit message: Go through and fix notation on RS485 wiring everywhere to use the standard A/B notation.
Parts:
- added R10, R11, R12, R13, R14, R15, R4, R5, R6, R7, R8, R9: 120ohm, rcl:R0805
- R1, R2, R3: device rcl:R1206 -> rcl:R0805
Connections:
- removed net CAM10D+: CAM10.2, U3.14
- removed net CAM10D-: CAM10.1, U3.13
- removed net CAM11D+: CAM11.2, U3.6
- removed net CAM11D-: CAM11.1, U3.5
- removed net CAM12D+: CAM12.2, U3.10
- removed net CAM12D-: CAM12.1, U3.11
- removed net CAM1D+: CAM1.2, U1.2
- removed net CAM1D-: CAM1.1, U1.3
- removed net CAM2D+: CAM2.2, U1.14
- removed net CAM2D-: CAM2.1, U1.13
- removed net CAM3D+: CAM3.2, U1.6
- removed net CAM3D-: CAM3.1, U1.5
- removed net CAM4D+: CAM4.2, U1.10
- removed net CAM4D-: CAM4.1, U1.11
- removed net CAM5D+: CAM5.2, U2.2
- removed net CAM5D-: CAM5.1, U2.3
- removed net CAM6D+: CAM6.2, U2.14
- removed net CAM6D-: CAM6.1, U2.13
- removed net CAM7D+: CAM7.2, U2.6
- removed net CAM7D-: CAM7.1, U2.5
- removed net CAM8D+: CAM8.2, U2.10
- removed net CAM8D-: CAM8.1, U2.11
- removed net CAM9D+: CAM9.2, U3.2
- removed net CAM9D-: CAM9.1, U3.3
- new net CAM10DA: CAM10.1, R13.1, U3.14
- new net CAM10DB: CAM10.2, R13.2, U3.13
- new net CAM11DA: CAM11.1, R14.1, U3.6
- new net CAM11DB: CAM11.2, R14.2, U3.5
- new net CAM12DA: CAM12.1, R15.1, U3.10
- new net CAM12DB: CAM12.2, R15.2, U3.11
- new net CAM1DA: CAM1.1, R4.1, U1.2
- new net CAM1DB: CAM1.2, R4.2, U1.3
- new net CAM2DA: CAM2.1, R5.1, U1.14
- new net CAM2DB: CAM2.2, R5.2, U1.13
- new net CAM3DA: CAM3.1, R6.1, U1.6
- new net CAM3DB: CAM3.2, R6.2, U1.5
- new net CAM4DA: CAM4.1, R7.1, U1.10
- new net CAM4DB: CAM4.2, R7.2, U1.11
- new net CAM5DA: CAM5.1, R8.1, U2.2
- new net CAM5DB: CAM5.2, R8.2, U2.3
- new net CAM6DA: CAM6.1, R9.1, U2.14
- new net CAM6DB: CAM6.2, R9.2, U2.13
- new net CAM7DA: CAM7.1, R10.1, U2.6
- new net CAM7DB: CAM7.2, R10.2, U2.5
- new net CAM8DA: CAM8.1, R11.1, U2.10
- new net CAM8DB: CAM8.2, R11.2, U2.11
- new net CAM9DA: CAM9.1, R12.1, U3.2
- new net CAM9DB: CAM9.2, R12.2, U3.3
Routing:
- net CAM12DB: track 0.00 -> 21.5 mm, vias 0 -> 1
- net CAM8DB: track 0.00 -> 21.5 mm, vias 0 -> 1
- net CAM4DB: track 0.00 -> 18.5 mm, vias 0 -> 1
- net CAM8DA: track 0.00 -> 16.4 mm
- net CAM12DA: track 0.00 -> 16.4 mm
- net CAM2DA: track 0.00 -> 16.4 mm
- net CAM10DA: track 0.00 -> 16.4 mm
- net CAM6DA: track 0.00 -> 16.4 mm
- net CAM4DA: track 0.00 -> 16.4 mm
- net CAM2DB: track 0.00 -> 16.4 mm
- net CAM10DB: track 0.00 -> 16.4 mm, vias 0 -> 1
- net CAM6DB: track 0.00 -> 16.4 mm, vias 0 -> 1
- net CAM12D+: track 14.8 -> 0.00 mm
- net CAM8D+: track 14.8 -> 0.00 mm
- net CAM12D-: track 14.8 -> 0.00 mm
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Other:
- board text added: "A B"

Commit message: Revisions to SMD version of controller board.  Create board for wireless tally.  Code revisions to sketch.
Routing:
- net MEGASDA1: track 33.3 -> 34.4 mm, vias 0 -> 1
- net MEGASCL1: track 33.3 -> 34.4 mm
Changed lines of the file:
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@@
 <drawing>
 <settings>
-<setting alwaysvectorfont="yes"/>
+<setting alwaysvectorfont="no"/>
 <setting verticaltext="up"/>
 </settings>
@@
 <contactref element="TALENT_DIM" pad="1"/>
 <contactref element="OP_DIM" pad="1"/>
-<via x="20.32" y="43.18" extent="1-16" drill="0.35"/>
 <contactref element="EXTPOWER" pad="1"/>
 <via x="68.58" y="33.02" extent="1-16" drill="0.35"/>
@@
 </signal>
 <signal name="MEGASDA1">
+<contactref element="I2C" pad="3"/>
+<wire x1="8.89" y1="24.13" x2="8.89" y2="21.59" width="0.1524" layer="1"/>
 <contactref element="J2" pad="SDA1"/>
-<contactref element="I2C" pad="3"/>
-<wire x1="8.89" y1="21.59" x2="8.89" y2="24.13" width="0.1524" layer="1"/>
-<wire x1="18.796" y1="34.036" x2="18.796" y2="50.8" width="0.1524" layer="1"/>
-<wire x1="8.89" y1="24.13" x2="18.796" y2="34.036" width="0.1524" layer="1"/>
+<via x="19.05" y="38.1" extent="1-16" drill="0.35"/>
+<wire x1="19.05" y1="38.1" x2="19.05" y2="34.29" width="0.1524" layer="1"/>
+<wire x1="19.05" y1="34.29" x2="8.89" y2="24.13" width="0.1524" layer="1"/>
+<wire x1="21.336" y1="50.8" x2="21.336" y2="41.656" width="0.1524" layer="16"/>
+<wire x1="19.05" y1="39.37" x2="19.05" y2="38.1" width="0.1524" layer="16"/>
+<wire x1="21.336" y1="41.656" x2="19.05" y2="39.37" width="0.1524" layer="16"/>
 </signal>
 <signal name="MEGASCL1">
-<contactref element="J2" pad="SCL1"/>
 <contactref element="I2C" pad="4"/>
 <wire x1="11.43" y1="21.59" x2="11.43" y2="24.13" width="0.1524" layer="1"/>
-<wire x1="21.336" y1="34.036" x2="21.336" y2="50.8" width="0.1524" layer="1"/>
 <wire x1="11.43" y1="24.13" x2="21.336" y2="34.036" width="0.1524" layer="1"/>
+<contactref element="J2" pad="SCL1"/>
+<wire x1="21.336" y1="39.624" x2="21.336" y2="34.036" width="0.1524" layer="1"/>
+<wire x1="18.796" y1="50.8" x2="18.796" y2="42.164" width="0.1524" layer="1"/>
+<wire x1="18.796" y1="42.164" x2="21.336" y2="39.624" width="0.1524" layer="1"/>
 </signal>
 <signal name="MEGA53">
