File: TallyController/EAGLE/tally-controller-shield-smd.sch (EAGLE design)
At the start: 40 parts, among them J2 Mega R3, U1 SN75174N, U2 SN75174N, U3 SN75174N

Commit message: Revisions to boards after working with initial prototypes.
- Update boards to use SMD components to help save on space.
- Redesign wireless receiver to use 3.3v logic to avoid using the Xbee breakout.
- Remove designs that aren't going to be used.
Parts:
- added C1: 1000uf, SparkFun-Capacitors:1000UF-RADIAL-5MM-25V-20%
- added SW1: B3U-1000P, Switch:B3U-1000P
Connections:
- net GND: now also C1.-, SW1.1
- net RESET: now also SW1.2
- net VCC: now also C1.+
Changed lines of the file:
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@@
 <layer number="56" name="wert" color="7" fill="1" visible="no" active="no"/>
 <layer number="57" name="tCAD" color="7" fill="1" visible="no" active="no"/>
+<layer number="59" name="tCarbon" color="7" fill="1" visible="no" active="no"/>
+<layer number="60" name="bCarbon" color="7" fill="1" visible="no" active="no"/>
+<layer number="88" name="SimResults" color="9" fill="1" visible="yes" active="yes"/>
+<layer number="89" name="SimProbes" color="9" fill="1" visible="yes" active="yes"/>
 <layer number="90" name="Modules" color="5" fill="1" visible="yes" active="yes"/>
 <layer number="91" name="Nets" color="2" fill="1" visible="yes" active="yes"/>
@@
 <layer number="97" name="Info" color="5" fill="1" visible="yes" active="yes"/>
 <layer number="98" name="Guide" color="6" fill="1" visible="yes" active="yes"/>
+<layer number="99" name="SpiceOrder" color="7" fill="1" visible="yes" active="yes"/>
 <layer number="100" name="Muster" color="7" fill="1" visible="no" active="no"/>
 <layer number="101" name="Patch_Top" color="12" fill="4" visible="yes" active="yes"/>
@@
 <layer number="111" name="LPC17xx" color="7" fill="1" visible="yes" active="yes"/>
 <layer number="112" name="tSilk" color="7" fill="1" visible="yes" active="yes"/>
+<layer number="113" name="IDFDebug" color="7" fill="1" visible="yes" active="yes"/>
+<layer number="114" name="Badge_Outline" color="7" fill="1" visible="yes" active="yes"/>
+<layer number="115" name="ReferenceISLANDS" color="7" fill="1" visible="yes" active="yes"/>
 <layer number="116" name="Patch_BOT" color="9" fill="4" visible="yes" active="yes"/>
+<layer number="118" name="Rect_Pads" color="7" fill="1" visible="yes" active="yes"/>
 <layer number="121" name="_tsilk" color="7" fill="1" visible="yes" active="yes"/>
 <layer number="122" name="_bsilk" color="7" fill="1" visible="yes" active="yes"/>
@@
 <layer number="127" name="_tValues" color="7" fill="1" visible="yes" active="yes"/>
 <layer number="128" name="_bValues" color="7" fill="1" visible="yes" active="yes"/>
+<layer number="129" name="Mask" color="7" fill="1" visible="yes" active="yes"/>
 <layer number="131" name="tAdjust" color="7" fill="1" visible="no" active="yes"/>
 <layer number="132" name="bAdjust" color="7" fill="1" visible="no" active="yes"/>
@@
 <layer number="223" name="223bmp" color="24" fill="1" visible="no" active="no"/>
 <layer number="224" name="224bmp" color="25" fill="1" visible="no" active="no"/>
+<layer number="225" name="225bmp" color="7" fill="1" visible="yes" active="yes"/>
+<layer number="226" name="226bmp" color="7" fill="1" visible="yes" active="yes"/>
+<layer number="227" name="227bmp" color="7" fill="1" visible="yes" active="yes"/>
+<layer number="228" name="228bmp" color="7" fill="1" visible="yes" active="yes"/>
+<layer number="229" name="229bmp" color="7" fill="1" visible="yes" active="yes"/>
+<layer number="230" name="230bmp" color="7" fill="1" visible="yes" active="yes"/>
+<layer number="231" name="231bmp" color="7" fill="1" visible="yes" active="yes"/>
 <layer number="248" name="Housing" color="7" fill="1" visible="yes" active="yes"/>
 <layer number="249" name="Edge" color="7" fill="1" visible="yes" active="yes"/>
@@
 <layer number="251" name="SMDround" color="7" fill="1" visible="no" active="no"/>
 <layer number="254" name="cooling" color="7" fill="1" visible="yes" active="yes"/>
+<layer number="255" name="routoute" color="7" fill="1" visible="yes" active="yes"/>
 </layers>
 <schematic xreflabel="%F%N/%S.%C%R" xrefpart="/%S.%C%R">
@@
 <part name="R14" library="rcl" library_urn="urn:adsk.eagle:library:334" deviceset="R-US_" device="R0805" package3d_urn="urn:adsk.eagle:package:23553/2" value="120ohm"/>
 <part name="R15" library="rcl" library_urn="urn:adsk.eagle:library:334" deviceset="R-US_" device="R0805" package3d_urn="urn:adsk.eagle:package:23553/2" value="120ohm"/>
+<part name="C1" library="SparkFun-Capacitors" library_urn="urn:adsk.eagle:library:510" deviceset="1000UF" device="-RADIAL-5MM-25V-20%" package3d_urn="urn:adsk.eagle:package:37412/1" value="1000uf"/>
+<part name="SW1" library="Switch" library_urn="urn:adsk.eagle:library:11396471" deviceset="B3U-1000P" device="" package3d_urn="urn:adsk.eagle:package:10899220/2"/>
 </parts>
 <sheets>
@@
 <attribute name="NAME" x="-34.29" y="31.9786" size="1.778" layer="95"/>
 <attribute name="VALUE" x="-34.29" y="27.178" size="1.778" layer="96"/>
+</instance>
+<instance part="C1" gate="G$1" x="-27.94" y="154.94" smashed="yes">
+<attribute name="NAME" x="-26.924" y="155.575" size="1.778" layer="95" font="vector"/>
+<attribute name="VALUE" x="-26.924" y="150.749" size="1.778" layer="96" font="vector"/>
+</instance>
+<instance part="SW1" gate="G$1" x="-38.1" y="7.62" smashed="yes">
+<attribute name="NAME" x="-43.18" y="11.176" size="1.778" layer="95"/>
+<attribute name="VALUE" x="-43.18" y="2.54" size="1.778" layer="96"/>
 </instance>
 </instances>
@@
 <label x="-73.66" y="154.94" size="1.778" layer="95"/>
 </segment>
+<segment>
+<pinref part="C1" gate="G$1" pin="-"/>
+<wire x1="-27.94" y1="149.86" x2="-38.1" y2="149.86" width="0.1524" layer="91"/>
+<label x="-38.1" y="149.86" size="1.778" layer="95"/>
+</segment>
+<segment>
+<wire x1="-48.26" y1="7.62" x2="-55.88" y2="7.62" width="0.1524" layer="91"/>
+<label x="-55.88" y="7.62" size="1.778" layer="95"/>
+<pinref part="SW1" gate="G$1" pin="1"/>
+</segment>
 </net>
 <net name="MEGASDA" class="0">
@@
 <wire x1="-119.38" y1="83.82" x2="-139.7" y2="83.82" width="0.1524" layer="91"/>
 </segment>
+<segment>
+<wire x1="-27.94" y1="7.62" x2="-22.86" y2="7.62" width="0.1524" layer="91"/>
+<label x="-27.94" y="7.62" size="1.778" layer="95"/>
+<pinref part="SW1" gate="G$1" pin="2"/>
+</segment>
 </net>
 <net name="VCC" class="0">
@@
 <label x="-73.66" y="152.4" size="1.778" layer="95"/>
 </segment>
-</net>
+<segment>
+<pinref part="C1" gate="G$1" pin="+"/>
+<wire x1="-27.94" y1="157.48" x2="-38.1" y2="157.48" width="0.1524" layer="91"/>
+<label x="-38.1" y="157.48" size="1.778" layer="95"/>
+</segment>
+</net>

Commit message: Add decoupling caps to shield.
Remove non-SMD version of shield (no-longer being worked on).
Parts:
- added C2, C3, C4, C5, C6, C7: (no value), Nordic_nRF:CAPACITOR_0805_N
Connections:
- net GND: now also C2.2, C3.2, C4.2, C5.2, C6.2, C7.2
- net VCC: now also C2.1, C3.1, C4.1, C5.1, C6.1, C7.1
Changed lines of the file:
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@@
 <layer number="115" name="ReferenceISLANDS" color="7" fill="1" visible="yes" active="yes"/>
 <layer number="116" name="Patch_BOT" color="9" fill="4" visible="yes" active="yes"/>
+<layer number="117" name="BACKMAAT1" color="7" fill="1" visible="yes" active="yes"/>
 <layer number="118" name="Rect_Pads" color="7" fill="1" visible="yes" active="yes"/>
+<layer number="119" name="KAP_TEKEN" color="7" fill="1" visible="yes" active="yes"/>
+<layer number="120" name="KAP_MAAT1" color="7" fill="1" visible="yes" active="yes"/>
 <layer number="121" name="_tsilk" color="7" fill="1" visible="yes" active="yes"/>
 <layer number="122" name="_bsilk" color="7" fill="1" visible="yes" active="yes"/>
@@
 <layer number="128" name="_bValues" color="7" fill="1" visible="yes" active="yes"/>
 <layer number="129" name="Mask" color="7" fill="1" visible="yes" active="yes"/>
+<layer number="130" name="SMDSTROOK" color="7" fill="1" visible="yes" active="yes"/>
 <layer number="131" name="tAdjust" color="7" fill="1" visible="no" active="yes"/>
 <layer number="132" name="bAdjust" color="7" fill="1" visible="no" active="yes"/>
+<layer number="133" name="bottom_silk" color="7" fill="1" visible="yes" active="yes"/>
 <layer number="144" name="Drill_legend" color="7" fill="1" visible="yes" active="yes"/>
 <layer number="150" name="Notes" color="7" fill="1" visible="no" active="yes"/>
@@
 <layer number="230" name="230bmp" color="7" fill="1" visible="yes" active="yes"/>
 <layer number="231" name="231bmp" color="7" fill="1" visible="yes" active="yes"/>
+<layer number="232" name="Eagle3D_PG2" color="7" fill="1" visible="yes" active="yes"/>
+<layer number="233" name="Eagle3D_PG3" color="7" fill="1" visible="yes" active="yes"/>
 <layer number="248" name="Housing" color="7" fill="1" visible="yes" active="yes"/>
 <layer number="249" name="Edge" color="7" fill="1" visible="yes" active="yes"/>
@@
 <part name="C1" library="SparkFun-Capacitors" library_urn="urn:adsk.eagle:library:510" deviceset="1000UF" device="-RADIAL-5MM-25V-20%" package3d_urn="urn:adsk.eagle:package:37412/1" value="1000uf"/>
 <part name="SW1" library="Switch" library_urn="urn:adsk.eagle:library:11396471" deviceset="B3U-1000P" device="" package3d_urn="urn:adsk.eagle:package:10899220/2"/>
+<part name="C2" library="Nordic_nRF" library_urn="urn:adsk.eagle:library:169009" deviceset="CAPACITOR" device="_0805_N" package3d_urn="urn:adsk.eagle:package:2593736/1"/>
+<part name="C3" library="Nordic_nRF" library_urn="urn:adsk.eagle:library:169009" deviceset="CAPACITOR" device="_0805_N" package3d_urn="urn:adsk.eagle:package:2593736/1"/>
+<part name="C4" library="Nordic_nRF" library_urn="urn:adsk.eagle:library:169009" deviceset="CAPACITOR" device="_0805_N" package3d_urn="urn:adsk.eagle:package:2593736/1"/>
+<part name="C5" library="Nordic_nRF" library_urn="urn:adsk.eagle:library:169009" deviceset="CAPACITOR" device="_0805_N" package3d_urn="urn:adsk.eagle:package:2593736/1"/>
+<part name="C6" library="Nordic_nRF" library_urn="urn:adsk.eagle:library:169009" deviceset="CAPACITOR" device="_0805_N" package3d_urn="urn:adsk.eagle:package:2593736/1"/>
+<part name="C7" library="Nordic_nRF" library_urn="urn:adsk.eagle:library:169009" deviceset="CAPACITOR" device="_0805_N" package3d_urn="urn:adsk.eagle:package:2593736/1"/>
 </parts>
 <sheets>
@@
 <attribute name="NAME" x="-43.18" y="11.176" size="1.778" layer="95"/>
 <attribute name="VALUE" x="-43.18" y="2.54" size="1.778" layer="96"/>
+</instance>
+<instance part="C2" gate="C$1" x="53.34" y="35.56" smashed="yes">
+<attribute name="NAME" x="54.864" y="35.941" size="1.778" layer="95"/>
+<attribute name="VALUE" x="54.864" y="30.861" size="1.778" layer="96"/>
+</instance>
+<instance part="C3" gate="C$1" x="58.42" y="35.56" smashed="yes">
+<attribute name="NAME" x="59.944" y="35.941" size="1.778" layer="95"/>
+<attribute name="VALUE" x="59.944" y="30.861" size="1.778" layer="96"/>
+</instance>
+<instance part="C4" gate="C$1" x="63.5" y="35.56" smashed="yes">
+<attribute name="NAME" x="65.024" y="35.941" size="1.778" layer="95"/>
+<attribute name="VALUE" x="65.024" y="30.861" size="1.778" layer="96"/>
+</instance>
+<instance part="C5" gate="C$1" x="68.58" y="35.56" smashed="yes">
+<attribute name="NAME" x="70.104" y="35.941" size="1.778" layer="95"/>
+<attribute name="VALUE" x="70.104" y="30.861" size="1.778" layer="96"/>
+</instance>
+<instance part="C6" gate="C$1" x="73.66" y="35.56" smashed="yes">
+<attribute name="NAME" x="75.184" y="35.941" size="1.778" layer="95"/>
+<attribute name="VALUE" x="75.184" y="30.861" size="1.778" layer="96"/>
+</instance>
+<instance part="C7" gate="C$1" x="78.74" y="35.56" smashed="yes">
+<attribute name="NAME" x="80.264" y="35.941" size="1.778" layer="95"/>
+<attribute name="VALUE" x="80.264" y="30.861" size="1.778" layer="96"/>
 </instance>
 </instances>
@@
 <pinref part="SW1" gate="G$1" pin="1"/>
 </segment>
+<segment>
+<pinref part="C2" gate="C$1" pin="2"/>
+<wire x1="53.34" y1="30.48" x2="53.34" y2="27.94" width="0.1524" layer="91"/>
+<wire x1="53.34" y1="27.94" x2="58.42" y2="27.94" width="0.1524" layer="91"/>
+<pinref part="C3" gate="C$1" pin="2"/>
+<wire x1="58.42" y1="27.94" x2="58.42" y2="30.48" width="0.1524" layer="91"/>
+<pinref part="C4" gate="C$1" pin="2"/>
+<wire x1="63.5" y1="30.48" x2="63.5" y2="27.94" width="0.1524" layer="91"/>
+<wire x1="63.5" y1="27.94" x2="58.42" y2="27.94" width="0.1524" layer="91"/>
+<junction x="58.42" y="27.94"/>
+<label x="58.42" y="25.4" size="1.778" layer="95"/>
+<pinref part="C5" gate="C$1" pin="2"/>
+<wire x1="68.58" y1="30.48" x2="68.58" y2="27.94" width="0.1524" layer="91"/>
+<wire x1="68.58" y1="27.94" x2="63.5" y2="27.94" width="0.1524" layer="91"/>
+<junction x="63.5" y="27.94"/>
+<pinref part="C6" gate="C$1" pin="2"/>
+<wire x1="73.66" y1="30.48" x2="73.66" y2="27.94" width="0.1524" layer="91"/>
+<wire x1="73.66" y1="27.94" x2="68.58" y2="27.94" width="0.1524" layer="91"/>
+<junction x="68.58" y="27.94"/>
+<pinref part="C7" gate="C$1" pin="2"/>
+<wire x1="78.74" y1="30.48" x2="78.74" y2="27.94" width="0.1524" layer="91"/>
+<wire x1="78.74" y1="27.94" x2="73.66" y2="27.94" width="0.1524" layer="91"/>
+<junction x="73.66" y="27.94"/>
+</segment>
 </net>
 <net name="MEGASDA" class="0">
@@
 <label x="-38.1" y="157.48" size="1.778" layer="95"/>
 </segment>
-</net>
+<segment>
+<pinref part="C2" gate="C$1" pin="1"/>
+<wire x1="53.34" y1="38.1" x2="53.34" y2="40.64" width="0.1524" layer="91"/>
+<wire x1="53.34" y1="40.64" x2="58.42" y2="40.64" width="0.1524" layer="91"/>
+<pinref part="C4" gate="C$1" pin="1"/>
+<wire x1="58.42" y1="40.64" x2="63.5" y2="40.64" width="0.1524" layer="91"/>
+<wire x1="63.5" y1="40.64" x2="63.5" y2="38.1" width="0.1524" layer="91"/>
+<pinref part="C3" gate="C$1" pin="1"/>
+<wire x1="58.42" y1="38.1" x2="58.42" y2="40.64" width="0.1524" layer="91"/>
+<junction x="58.42" y="40.64"/>
+<label x="58.42" y="40.64" size="1.778" layer="95"/>
+<pinref part="C5" gate="C$1" pin="1"/>
+<wire x1="68.58" y1="38.1" x2="68.58" y2="40.64" width="0.1524" layer="91"/>
+<wire x1="68.58" y1="40.64" x2="63.5" y2="40.64" width="0.1524" layer="91"/>
+<junction x="63.5" y="40.64"/>
+<pinref part="C6" gate="C$1" pin="1"/>
+<wire x1="73.66" y1="38.1" x2="73.66" y2="40.64" width="0.1524" layer="91"/>
+<wire x1="73.66" y1="40.64" x2="68.58" y2="40.64" width="0.1524" layer="91"/>
+<junction x="68.58" y="40.64"/>
+<pinref part="C7" gate="C$1" pin="1"/>
+<wire x1="78.74" y1="38.1" x2="78.74" y2="40.64" width="0.1524" layer="91"/>
+<wire x1="78.74" y1="40.64" x2="73.66" y2="40.64" width="0.1524" layer="91"/>
+<junction x="73.66" y="40.64"/>
+</segment>
+</net>

Commit message: Add optional AREF jumper.  Remove unused nets.
Parts:
- added AREF: 0ohm, BeagleBone_Black_Wireless:R-US_0204/2V
- C2, C3, C4, C5, C6, C7: value (none) -> 1uf
Connections:
- removed net 5V@1: J2.5V@1
- removed net 5V@2: J2.5V@2
- removed net IOREF: J2.IOREF
- removed net MEGA10: J2.10
- removed net MEGA2: J2.2
- removed net MEGA23: J2.23
- removed net MEGA25: J2.25
- removed net MEGA27: J2.27
- removed net MEGA29: J2.29
- removed net MEGA3: J2.3
- removed net MEGA30: J2.30
- removed net MEGA31: J2.31
- removed net MEGA32: J2.32
- removed net MEGA33: J2.33
- removed net MEGA34: J2.34
- removed net MEGA35: J2.35
- removed net MEGA36: J2.36
- removed net MEGA37: J2.37
- removed net MEGA39: J2.39
- removed net MEGA4: J2.4
- removed net MEGA41: J2.41
- removed net MEGA43: J2.43
- removed net MEGA45: J2.45
- removed net MEGA46: J2.46
- removed net MEGA47: J2.47
- removed net MEGA48: J2.48
- removed net MEGA49: J2.49
- removed net MEGA53: J2.53
- removed net MEGA9: J2.9
- removed net MEGAA10: J2.A10
- removed net MEGAA11: J2.A11
- removed net MEGAA12: J2.A12
- removed net MEGAA13: J2.A13
- removed net MEGAA14: J2.A14
- removed net MEGAA15: J2.A15
- removed net MEGAA3: J2.A3
- removed net MEGAA4: J2.A4
- removed net MEGAA5: J2.A5
- removed net MEGAA6: J2.A6
- removed net MEGAA7: J2.A7
- removed net MEGAA8: J2.A8
- removed net MEGAA9: J2.A9
- removed net MEGAMISO: J2.50
- removed net MEGAMOSI: J2.51
- removed net MEGARX0: J2.0(RX0)
- removed net MEGARX3: J2.15(RX3)
- removed net MEGASCL: J2.21(SCL)
- removed net MEGASCLK: J2.52
- removed net MEGASDA: J2.20(SDA)
- removed net MEGATX0: J2.1(TX0)
- removed net MEGATX3: J2.14(TX3)
- removed net VIN: J2.VIN
- new net AREF: AREF.1, J2.AREF
- net VCC: now also AREF.2
